File: board2.sch (EAGLE design)
At the start: 45 parts, among them J1 U.FL, X1 26MHz 10pF 10ppm -20C +70C

Commit message: notes n no backup
Other:
- note added: "NOTES"
- note added: "Ordered 6/28/2015 OSHPark"
Changed lines of the file:
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@@
 <plain>
 <text x="170.18" y="132.08" size="1.27" layer="95" font="vector">LIPO Battery</text>
+<text x="238.76" y="101.6" size="5.08" layer="94" ratio="15">Ordered 6/28/2015 OSHPark</text>
+<text x="284.48" y="127" size="6.4516" layer="94" ratio="15">NOTES</text>
 </plain>
 <instances>
@@
 </segment>
 </net>
+<net name="N$11" class="0">
+<segment>
+<wire x1="231.14" y1="-71.12" x2="358.14" y2="-71.12" width="1.778" layer="91"/>
+<wire x1="358.14" y1="-71.12" x2="358.14" y2="144.78" width="1.778" layer="91"/>
+<wire x1="358.14" y1="144.78" x2="231.14" y2="144.78" width="1.778" layer="91"/>
+<wire x1="231.14" y1="144.78" x2="231.14" y2="-71.12" width="1.778" layer="91"/>
+</segment>
+</net>

Commit message: New Notes
Other:
- note added: "All other traces checked, thickened and angled."
- note added: "New CC1110 Lib New BLE113-A Lib New TPS63031 Lib New 0915bM15A0001 Lib"
- note added: "Traces under debug connectors fixed"
- note added: "USB Switched (Same Position) C4 Moved Down Lipo Moved Up"
Changed lines of the file:
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@@
 <plain>
 <text x="170.18" y="132.08" size="1.27" layer="95" font="vector">LIPO Battery</text>
-<text x="238.76" y="101.6" size="5.08" layer="94" ratio="15">Ordered 6/28/2015 OSHPark</text>
+<text x="238.76" y="-63.5" size="5.08" layer="94" ratio="15">Ordered 6/28/2015 OSHPark</text>
 <text x="284.48" y="127" size="6.4516" layer="94" ratio="15">NOTES</text>
+<text x="241.3" y="86.36" size="5.08" layer="94" ratio="15">New CC1110 Lib
+New BLE113-A Lib
+New TPS63031 Lib
+New 0915bM15A0001 Lib</text>
+<text x="241.3" y="55.88" size="5.08" layer="94" ratio="15">USB Switched (Same Position)
+C4 Moved Down
+Lipo Moved Up</text>
+<text x="241.3" y="33.02" size="5.08" layer="94" ratio="15">Traces under debug
+connectors fixed</text>
+<text x="241.3" y="10.16" size="5.08" layer="94" ratio="15">All other traces checked,
+thickened and angled.</text>
 </plain>
 <instances>
@@
 <net name="N$11" class="0">
 <segment>
-<wire x1="231.14" y1="-71.12" x2="358.14" y2="-71.12" width="1.778" layer="91"/>
-<wire x1="358.14" y1="-71.12" x2="358.14" y2="144.78" width="1.778" layer="91"/>
-<wire x1="358.14" y1="144.78" x2="231.14" y2="144.78" width="1.778" layer="91"/>
+<wire x1="231.14" y1="-71.12" x2="368.3" y2="-71.12" width="1.778" layer="91"/>
+<wire x1="368.3" y1="-71.12" x2="368.3" y2="144.78" width="1.778" layer="91"/>
+<wire x1="368.3" y1="144.78" x2="231.14" y2="144.78" width="1.778" layer="91"/>
 <wire x1="231.14" y1="144.78" x2="231.14" y2="-71.12" width="1.778" layer="91"/>
 </segment>
@@
 </schematic>
 </drawing>
+<compatibility>
+<note version="6.3" minversion="6.2.2" severity="warning">
+Since Version 6.2.2 text objects can contain more than one line,
+which will not be processed correctly with this version.
+</note>
+</compatibility>
 </eagle>
